File: Sega CD RAM Cart.sch (KiCad schematic (older format))
At the start: 27 parts, among them J1 Genesis_Edge_Connector, U1 74LS30, U2 IS61C5128AS-25QLI, U3 74LS30, U4 74LS138, U5 74LS32, U6 74LS74, U7 74LS245

Commit message: Finalizing design.
Parts:
- added H1, H2: MountingHole, Sega CD RAM Cart:MountingHole_6.2mm, symbol Mechanical:MountingHole
Changed lines of the file:
@@
 L power:VBUS #PWR0109
 U 1 1 617FBDD3
-P 1150 7550
-F 0 "#PWR0109" H 1150 7400 50  0001 C CNN
-F 1 "VBUS" H 1165 7723 50  0000 C CNN
-F 2 "" H 1150 7550 50  0001 C CNN
-F 3 "" H 1150 7550 50  0001 C CNN
-	1    1150 7550
+P 750 7100
+F 0 "#PWR0109" H 750 6950 50  0001 C CNN
+F 1 "VBUS" H 765 7273 50  0000 C CNN
+F 2 "" H 750 7100 50  0001 C CNN
+F 3 "" H 750 7100 50  0001 C CNN
+	1    750  7100
 	-1   0    0    1
 $EndComp
@@
 L power:PWR_FLAG #FLG0103
 U 1 1 617FD675
-P 1150 7550
-F 0 "#FLG0103" H 1150 7625 50  0001 C CNN
-F 1 "PWR_FLAG" H 1150 7723 50  0000 C CNN
-F 2 "" H 1150 7550 50  0001 C CNN
-F 3 "~" H 1150 7550 50  0001 C CNN
-	1    1150 7550
+P 750 7100
+F 0 "#FLG0103" H 750 7175 50  0001 C CNN
+F 1 "PWR_FLAG" H 750 7273 50  0000 C CNN
+F 2 "" H 750 7100 50  0001 C CNN
+F 3 "~" H 750 7100 50  0001 C CNN
+	1    750  7100
 	1    0    0    -1
 $EndComp
@@
 	2250 1150 2250 1700
 NoConn ~ 5300 4500
+$Comp
+L Mechanical:MountingHole H1
+U 1 1 61200889
+P 1050 7450
+F 0 "H1" H 1150 7496 50  0000 L CNN
+F 1 "MountingHole" H 1150 7405 50  0000 L CNN
+F 2 "Sega CD RAM Cart:MountingHole_6.2mm" H 1050 7450 50  0001 C CNN
+F 3 "~" H 1050 7450 50  0001 C CNN
+	1    1050 7450
+	1    0    0    -1
+$EndComp
+$Comp
+L Mechanical:MountingHole H2
+U 1 1 612020AB
+P 1050 7650
+F 0 "H2" H 1150 7696 50  0000 L CNN
+F 1 "MountingHole" H 1150 7605 50  0000 L CNN
+F 2 "Sega CD RAM Cart:MountingHole_6.2mm" H 1050 7650 50  0001 C CNN
+F 3 "~" H 1050 7650 50  0001 C CNN
+	1    1050 7650
+	1    0    0    -1
+$EndComp
 $EndSCHEMATC

Commit message: More cleanup.
Boards approaching final rev. Added OSHW logos & other stuff.
Parts:
- removed R2, R3, R4, R5, R6, R7, R8, R9: 1K, Resistor_SMD:R_0805_2012Metric_Pad1.20x1.40mm_HandSolder, symbol Device:R
- BT1: symbol Sega~Genesis:Battery_Cell -> Sega_Genesis:Battery_Cell
- C8: value 22uF 16v -> 22uF 25v; Digikey PN UMV1C220MFD -> 25ML22MEFC5X5
- D1: value BAT5405E -> MMBD1204; symbol Sega~Genesis:BAT5405E -> Sega_Genesis:BAT5405E; Category Discrete Semiconductor Products -> (none); DK_Datasheet_Link https://www.diodes.com/assets/Datasheets/ds11005.pdf -> (none); DK_Detail_Page /product-detail/en/diodes-incorporated/BAT54C-7-F/BAT54C-FD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 -> (none); Description DIODE ARRAY SCHOTTKY 30V SOT23-3 -> (none); Digi-Key_PN BAT54C-FDICT-ND -> (none); Digikey PN (none) -> MMBD1204CT-ND; Family Diodes - Rectifiers - Arrays -> (none); MPN BAT54C-7-F -> (none); Manufacturer Diodes Incorporated -> (none); Status Active -> (none)
- J1: symbol Sega~Genesis:Genesis_Edge_Connector -> Sega_Genesis:Genesis_Edge_Connector
Connections:
- wire segments 176 -> 164
- no-connect marks 38 -> 33
Other:
- moved on the sheet: C7, U4

Commit message: Board tweaks.
U5D OR Gate inputs tied up so they don't float. No other changes.
Parts:
- added unit 4 of U5
Connections:
- wire segments 164 -> 167
- no-connect marks 33 -> 34
Changed lines of the file:
@@
 	8300 700  8550 700
 Connection ~ 8550 700
+$Comp
+L 74xx:74LS32 U5
+U 4 1 612C0675
+P 3150 6500
+F 0 "U5" H 3150 6825 50  0000 C CNN
+F 1 "74LS32" H 3150 6734 50  0000 C CNN
+F 2 "" H 3150 6500 50  0001 C CNN
+F 3 "http://www.ti.com/lit/gpn/sn74LS32" H 3150 6500 50  0001 C CNN
+	4    3150 6500
+	1    0    0    -1
+$EndComp
+$Comp
+L power:+5V #PWR0112
+U 1 1 612F1CBB
+P 2650 6400
+F 0 "#PWR0112" H 2650 6250 50  0001 C CNN
+F 1 "+5V" H 2665 6573 50  0000 C CNN
+F 2 "" H 2650 6400 50  0001 C CNN
+F 3 "" H 2650 6400 50  0001 C CNN
+	1    2650 6400
+	1    0    0    -1
+$EndComp
+NoConn ~ 3450 6500
+$Comp
+L power:GND #PWR?
+U 1 1 613115A5
+P 2850 6300
+F 0 "#PWR?" H 2850 6050 50  0001 C CNN
+F 1 "GND" H 2855 6127 50  0000 C CNN
+F 2 "" H 2850 6300 50  0001 C CNN
+F 3 "" H 2850 6300 50  0001 C CNN
+	1    2850 6300
+	-1   0    0    1
+$EndComp
+Wire Wire Line
+	2650 6600 2650 6400
+Wire Wire Line
+	2650 6600 2850 6600
+Wire Wire Line
+	2850 6300 2850 6400
 $EndSCHEMATC

Commit message: Board Updates (+Board tested!)
Removed unneeded files, fixed A20/A22 swap @ U4. Boards tested working today after cut & jumper on the real PCB's.
Changed lines of the file:
@@
 	8050 1550 7600 1550
 Text Label 7800 1350 0    50   ~ 0
-A22
+A20
 Text Label 7800 1450 0    50   ~ 0
 A21
 Text Label 7800 1550 0    50   ~ 0
-A20
+A22
 $Comp
 L 74xx:74LS74 U6
@@
 NoConn ~ 3450 6500
 $Comp
-L power:GND #PWR?
+L power:GND #PWR0113
 U 1 1 613115A5
 P 2850 6300
-F 0 "#PWR?" H 2850 6050 50  0001 C CNN
+F 0 "#PWR0113" H 2850 6050 50  0001 C CNN
 F 1 "GND" H 2855 6127 50  0000 C CNN
 F 2 "" H 2850 6300 50  0001 C CNN

Commit message: BOM Fix
Realized I specified a 1206 resistor instead of 0805. Fixed the BOM. Also added an HTML exported BOM for easy reading.
Parts:
- R1: Digikey PN CRGCQ1206J1K0 -> RMCF0805FT1K00
- U5: footprint (none) -> digikey-footprints:SOIC-14_W3.9mm; Digikey PN (none) -> SN74LS32DR
Changed lines of the file:
@@
 F 1 "IS61C5128AS-25QLI" H 3400 4390 50  0000 C CNN
 F 2 "Package_SO:SSOP-32_11.305x20.495mm_P1.27mm" H 2900 4150 50  0001 C CNN
-F 3 "http://www.issi.com/WW/pdf/61-64C5128AL.pdf" H 3400 3000 50  0001 C CNN
+F 3 "" H 3400 3000 50  0001 C CNN
 F 4 "IS61C5128AS-25QLI" H 3400 3000 50  0001 C CNN "Digikey PN"
 	1    3400 3000
@@
 F 1 "74LS30" H 8500 4200 50  0000 C CNN
 F 2 "digikey-footprints:SOIC-14_W3.9mm" H 8500 4000 50  0001 C CNN
-F 3 "http://www.ti.com/lit/gpn/sn74LS30" H 8500 4000 50  0001 C CNN
+F 3 "" H 8500 4000 50  0001 C CNN
 F 4 "SN74LS30DR" H 8500 4000 50  0001 C CNN "Digikey PN"
 	1    8500 4000
@@
 F 1 "74LS30" H 3650 7000 50  0000 L CNN
 F 2 "digikey-footprints:SOIC-14_W3.9mm" H 3800 7050 50  0001 C CNN
-F 3 "http://www.ti.com/lit/gpn/sn74LS30" H 3800 7050 50  0001 C CNN
+F 3 "" H 3800 7050 50  0001 C CNN
 F 4 "SN74LS30DR" H 3800 7050 50  0001 C CNN "Digikey PN"
 	2    3800 7050
@@
 F 1 "74LS30" H 4500 7000 50  0000 L CNN
 F 2 "digikey-footprints:SOIC-14_W3.9mm" H 4650 7050 50  0001 C CNN
-F 3 "http://www.ti.com/lit/gpn/sn74LS30" H 4650 7050 50  0001 C CNN
+F 3 "" H 4650 7050 50  0001 C CNN
 F 4 "SN74LS30DR" H 4650 7050 50  0001 C CNN "Digikey PN"
 	2    4650 7050
@@
 F 1 "74LS30" H 8500 3300 50  0000 C CNN
 F 2 "digikey-footprints:SOIC-14_W3.9mm" H 8500 3100 50  0001 C CNN
-F 3 "http://www.ti.com/lit/gpn/sn74LS30" H 8500 3100 50  0001 C CNN
+F 3 "" H 8500 3100 50  0001 C CNN
 F 4 "SN74LS30DR" H 8500 3100 50  0001 C CNN "Digikey PN"
 	1    8500 3100
@@
 F 1 "74LS32" H 9200 3734 50  0000 C CNN
 F 2 "digikey-footprints:SOIC-14_W3.9mm" H 9200 3500 50  0001 C CNN
-F 3 "http://www.ti.com/lit/gpn/sn74LS32" H 9200 3500 50  0001 C CNN
+F 3 "" H 9200 3500 50  0001 C CNN
 F 4 "SN74LS32DR" H 9200 3500 50  0001 C CNN "Digikey PN"
 	1    9200 3500
@@
 F 1 "74LS32" H 9900 2734 50  0000 C CNN
 F 2 "digikey-footprints:SOIC-14_W3.9mm" H 9900 2500 50  0001 C CNN
-F 3 "http://www.ti.com/lit/gpn/sn74LS32" H 9900 2500 50  0001 C CNN
+F 3 "" H 9900 2500 50  0001 C CNN
 F 4 "SN74LS32DR" H 9900 2500 50  0001 C CNN "Digikey PN"
 	2    9900 2500
@@
 F 1 "74LS74" H 8450 5640 50  0000 C CNN
 F 2 "digikey-footprints:SOIC-14_W3.9mm" H 8450 5250 50  0001 C CNN
-F 3 "74xx/74hc_hct74.pdf" H 8450 5250 50  0001 C CNN
+F 3 "" H 8450 5250 50  0001 C CNN
 F 4 "SN74LS74ADR" H 8450 5250 50  0001 C CNN "Digikey PN"
 	1    8450 5250
@@
 F 1 "74LS74" H 5350 7000 50  0000 L CNN
 F 2 "digikey-footprints:SOIC-14_W3.9mm" H 5500 7050 50  0001 C CNN
-F 3 "74xx/74hc_hct74.pdf" H 5500 7050 50  0001 C CNN
+F 3 "" H 5500 7050 50  0001 C CNN
 F 4 "SN74LS74ADR" H 5500 7050 50  0001 C CNN "Digikey PN"
 	3    5500 7050
@@
 F 1 "74LS32" H 6150 7000 50  0000 L CNN
 F 2 "digikey-footprints:SOIC-14_W3.9mm" H 6300 7050 50  0001 C CNN
-F 3 "http://www.ti.com/lit/gpn/sn74LS32" H 6300 7050 50  0001 C CNN
+F 3 "" H 6300 7050 50  0001 C CNN
 F 4 "SN74LS32DR" H 6300 7050 50  0001 C CNN "Digikey PN"
 	5    6300 7050
@@
 F 1 "74LS32" H 9350 5684 50  0000 C CNN
 F 2 "digikey-footprints:SOIC-14_W3.9mm" H 9350 5450 50  0001 C CNN
-F 3 "http://www.ti.com/lit/gpn/sn74LS32" H 9350 5450 50  0001 C CNN
+F 3 "" H 9350 5450 50  0001 C CNN
 F 4 "SN74LS32DR" H 9350 5450 50  0001 C CNN "Digikey PN"
 	3    9350 5450
@@
 F 1 "0.1uF" V 8950 700 50  0000 C CNN
 F 2 "Capacitor_SMD:C_1206_3216Metric_Pad1.33x1.80mm_HandSolder" H 8738 550 50  0001 C CNN
-F 3 "~" H 8700 700 50  0001 C CNN
+F 3 "" H 8700 700 50  0001 C CNN
 F 4 "C1206C104K4RACTU" H 8700 700 50  0001 C CNN "Digikey PN"
 	1    8700 700
@@
 F 1 "0.1uF" H 2765 1455 50  0000 L CNN
 F 2 "Capacitor_SMD:C_1206_3216Metric_Pad1.33x1.80mm_HandSolder" H 2688 1350 50  0001 C CNN
-F 3 "~" H 2650 1500 50  0001 C CNN
+F 3 "" H 2650 1500 50  0001 C CNN
 F 4 "C1206C104K4RACTU" H 2650 1500 50  0001 C CNN "Digikey PN"
 	1    2650 1500
@@
 F 1 "0.1uF" H 6815 6655 50  0000 L CNN
 F 2 "Capacitor_SMD:C_1206_3216Metric_Pad1.33x1.80mm_HandSolder" H 6738 6550 50  0001 C CNN
-F 3 "~" H 6700 6700 50  0001 C CNN
+F 3 "" H 6700 6700 50  0001 C CNN
 F 4 "C1206C104K4RACTU" H 6700 6700 50  0001 C CNN "Digikey PN"
 	1    6700 6700
@@
 F 1 "0.1uF" H 5965 6755 50  0000 L CNN
 F 2 "Capacitor_SMD:C_1206_3216Metric_Pad1.33x1.80mm_HandSolder" H 5888 6650 50  0001 C CNN
-F 3 "~" H 5850 6800 50  0001 C CNN
+F 3 "" H 5850 6800 50  0001 C CNN
 F 4 "C1206C104K4RACTU" H 5850 6800 50  0001 C CNN "Digikey PN"
 	1    5850 6800
@@
 F 1 "0.1uF" H 5165 6655 50  0000 L CNN
 F 2 "Capacitor_SMD:C_1206_3216Metric_Pad1.33x1.80mm_HandSolder" H 5088 6550 50  0001 C CNN
-F 3 "~" H 5050 6700 50  0001 C CNN
+F 3 "" H 5050 6700 50  0001 C CNN
 F 4 "C1206C104K4RACTU" H 5050 6700 50  0001 C CNN "Digikey PN"
 	1    5050 6700
@@
 F 1 "0.1uF" H 4315 6655 50  0000 L CNN
 F 2 "Capacitor_SMD:C_1206_3216Metric_Pad1.33x1.80mm_HandSolder" H 4238 6550 50  0001 C CNN
-F 3 "~" H 4200 6700 50  0001 C CNN
+F 3 "" H 4200 6700 50  0001 C CNN
 F 4 "C1206C104K4RACTU" H 4200 6700 50  0001 C CNN "Digikey PN"
 	1    4200 6700
@@
 F 1 "1K" V 1434 1050 50  0000 C CNN
 F 2 "Resistor_SMD:R_0805_2012Metric_Pad1.20x1.40mm_HandSolder" V 1480 1050 50  0001 C CNN
-F 3 "~" H 1550 1050 50  0001 C CNN
-F 4 "CRGCQ1206J1K0" H 1550 1050 50  0001 C CNN "Digikey PN"
+F 3 "" H 1550 1050 50  0001 C CNN
+F 4 "RMCF0805FT1K00" H 1550 1050 50  0001 C CNN "Digikey PN"
 	1    1550 1050
 	0    1    1    0
@@
 F 1 "Battery_Cell" H 1018 1255 50  0000 L CNN
 F 2 "BU2450SM:BAT_BU2450SM-JJ-G" V 900 1310 50  0001 C CNN
-F 3 "~" V 900 1310 50  0001 C CNN
+F 3 "" V 900 1310 50  0001 C CNN
 F 4 "BU2450SM-JJ-GTR" H 900 1250 50  0001 C CNN "Digikey PN"
 	1    900  1250
@@
 F 1 "74LS74" H 3100 7690 50  0000 C CNN
 F 2 "digikey-footprints:SOIC-14_W3.9mm" H 3100 7300 50  0001 C CNN
-F 3 "74xx/74hc_hct74.pdf" H 3100 7300 50  0001 C CNN
+F 3 "" H 3100 7300 50  0001 C CNN
 F 4 "SN74LS74ADR" H 3100 7300 50  0001 C CNN "Digikey PN"
 	2    3100 7300
@@
 F 1 "74LS138" H 8500 1600 50  0000 C CNN
 F 2 "digikey-footprints:SOIC-16_W3.90mm" H 8550 1650 50  0001 C CNN
-F 3 "http://www.ti.com/lit/gpn/sn74LS138" H 8550 1650 50  0001 C CNN
+F 3 "" H 8550 1650 50  0001 C CNN
 F 4 "SN74LS138DR" H 8550 1650 50  0001 C CNN "Digikey PN"
 	1    8550 1650
@@
 F 1 "22uF 25v" H 2250 7300 50  0000 L CNN
 F 2 "Capacitor_THT:CP_Radial_D5.0mm_P2.00mm" H 2188 7200 50  0001 C CNN
-F 3 "~" H 2150 7350 50  0001 C CNN
+F 3 "" H 2150 7350 50  0001 C CNN
 F 4 "25ML22MEFC5X5" H 2150 7350 50  0001 C CNN "Digikey PN"
 	1    2150 7350
@@
 F 1 "0.1uF" H 1865 4105 50  0000 L CNN
 F 2 "Capacitor_SMD:C_1206_3216Metric_Pad1.33x1.80mm_HandSolder" H 1788 4000 50  0001 C CNN
-F 3 "~" H 1750 4150 50  0001 C CNN
+F 3 "" H 1750 4150 50  0001 C CNN
 F 4 "C1206C104K4RACTU" H 1750 4150 50  0001 C CNN "Digikey PN"
 	1    1750 4150
@@
 F 1 "74LS245" H 1600 4850 50  0000 C CNN
 F 2 "digikey-footprints:SSOP-20_W5.3mm" H 1600 5150 50  0001 C CNN
-F 3 "http://www.ti.com/lit/gpn/sn74LS245" H 1600 5150 50  0001 C CNN
+F 3 "" H 1600 5150 50  0001 C CNN
 F 4 "SN74LS245DBR" H 1600 5150 50  0001 C CNN "Digikey PN"
 	1    1600 5150
@@
 F 1 "MountingHole" H 1150 7405 50  0000 L CNN
 F 2 "Sega CD RAM Cart:MountingHole_6.2mm" H 1050 7450 50  0001 C CNN
-F 3 "~" H 1050 7450 50  0001 C CNN
+F 3 "" H 1050 7450 50  0001 C CNN
 	1    1050 7450
 	1    0    0    -1
@@
 F 1 "MountingHole" H 1150 7605 50  0000 L CNN
 F 2 "Sega CD RAM Cart:MountingHole_6.2mm" H 1050 7650 50  0001 C CNN
-F 3 "~" H 1050 7650 50  0001 C CNN
+F 3 "" H 1050 7650 50  0001 C CNN
 	1    1050 7650
 	1    0    0    -1
@@
 F 0 "U5" H 3150 6825 50  0000 C CNN
 F 1 "74LS32" H 3150 6734 50  0000 C CNN
-F 2 "" H 3150 6500 50  0001 C CNN
-F 3 "http://www.ti.com/lit/gpn/sn74LS32" H 3150 6500 50  0001 C CNN
+F 2 "digikey-footprints:SOIC-14_W3.9mm" H 3150 6500 50  0001 C CNN
+F 3 "" H 3150 6500 50  0001 C CNN
+F 4 "SN74LS32DR" H 3150 6500 50  0001 C CNN "Digikey PN"
 	4    3150 6500
 	1    0    0    -1
