File: Sega CD RAM Cart.kicad_pcb (KiCad board)
At the start: 2 copper layers, 83.8 x 61.5 mm, 27 parts, among them J1 Genesis_Edge_Connector, U1 74LS30, U2 IS61C5128AS-25QLI, U3 74LS30, U4 74LS138, U5 74LS32, U6 74LS74, U7 74LS245

Commit message: Finalizing design.
Parts:
- added H1: MountingHole, Sega CD RAM Cart:MountingHole_6.2mm, F.Cu at (90.5, 131.7)
- added H2: MountingHole, Sega CD RAM Cart:MountingHole_6.2mm, F.Cu at (160.3, 131.7)
Other:
- board text added: "Sega CD Back-up RAM Cart (4Mbit) v1.0 Designed by WindDrake with help from Officer_Skidmark Based on l_oliveira's original research github.com/WindDrake/SegaCD_Ramcart"
- board text removed: "Sega CD Back-up RAM Cart (4Mbit) Designed by WindDrake With help from Officer_Skidmark"

Commit message: More cleanup.
Boards approaching final rev. Added OSHW logos & other stuff.
Parts:
- removed R2, R3, R4, R5, R6, R7, R8, R9: 1K, Resistor_SMD:R_0805_2012Metric_Pad1.20x1.40mm_HandSolder
- added REF**: OSHW-Logo2_14.6x12mm_SilkScreen, Symbol:OSHW-Logo2_14.6x12mm_SilkScreen, B.Cu at (146.3, 127.1)
- added REF**: Symbol_CreativeCommonsPublicDomain_SilkScreenTop_Small, Symbol:Symbol_CreativeCommonsPublicDomain_SilkScreenTop_Small, B.Cu at (108.3, 108.2)
- added REF**: KiCad-Logo2_12mm_SilkScreen, Symbol:KiCad-Logo2_12mm_SilkScreen, B.Cu at (150.1, 111.0)
- C8: value 22uF 16v -> 22uF 25v
- D1: value BAT5405E -> MMBD1204
- moved C7 10.7 mm to (143.9, 138.2), turned to 270 degrees
- moved BT1 4.02 mm to (142.7, 119.2)
- moved C5 2.81 mm to (130.1, 132.8), turned to 0 degrees
Connections:
- U7 pad 11: Net-(R3-Pad2) -> GND
- U7 pad 12: Net-(R5-Pad2) -> GND
- U7 pad 13: Net-(R4-Pad2) -> GND
- U7 pad 14: Net-(R7-Pad2) -> GND
- U7 pad 15: Net-(R8-Pad2) -> GND
- U7 pad 16: Net-(R6-Pad1) -> +5V
- U7 pad 17: Net-(R2-Pad1) -> +5V
- U7 pad 18: Net-(R9-Pad2) -> GND
- U7 pad 5: Net-(U7-Pad5) -> GND
- U7 pad 6: Net-(U7-Pad6) -> GND
- U7 pad 7: Net-(U7-Pad7) -> GND
- U7 pad 8: Net-(U7-Pad8) -> GND
- U7 pad 9: Net-(U7-Pad9) -> GND
Routing:
- net Net-(R3-Pad2): track 15.5 -> 0.00 mm
- net Net-(R5-Pad2): track 12.9 -> 0.02 mm
- net Net-(R8-Pad2): track 11.3 -> 0.00 mm
- net Net-(R6-Pad1): track 10.9 -> 0.00 mm
- net Net-(R4-Pad2): track 9.40 -> 0.00 mm
- net GND: track 87.9 -> 79.2 mm, vias 23 -> 45
- net +5V: track 299.1 -> 291.4 mm
- net Net-(R2-Pad1): track 7.72 -> 0.00 mm
- net /A9: track 51.3 -> 58.6 mm, vias 2 -> 0
- net /D7: track 48.1 -> 54.1 mm
- net Net-(R7-Pad2): track 5.64 -> 0.00 mm
- net /A14: track 53.3 -> 48.7 mm
- net /A1: track 31.0 -> 35.3 mm
- net /A6: track 41.9 -> 45.8 mm
- net Net-(R9-Pad2): track 3.72 -> 0.00 mm
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
Commit message: Last Rev - PCB's Ordered
Full 1.0 revision is complete. PCB's ordered today through OSHPark.
Routing:
- net +5V: track 291.4 -> 290.1 mm
- net /TREN: track 22.0 -> 23.0 mm
- net /A16: track 72.7 -> 72.0 mm
- net GND: track 79.2 -> 79.5 mm, vias 45 -> 51

Commit message: Board tweaks.
U5D OR Gate inputs tied up so they don't float. No other changes.
Connections:
- U5 pad 11: (no net) -> Net-(U5-Pad11)
- U5 pad 12: (no net) -> GND
- U5 pad 13: (no net) -> +5V
Routing:
- net GND: track 79.5 -> 81.9 mm
- net +5V: track 290.1 -> 291.4 mm

Commit message: Board Updates (+Board tested!)
Removed unneeded files, fixed A20/A22 swap @ U4. Boards tested working today after cut & jumper on the real PCB's.
Connections:
- U4 pad 1: /A22 -> /A20
- U4 pad 3: /A20 -> /A22
Routing:
- net /A22: track 47.0 -> 50.2 mm
- net /A20: track 51.7 -> 51.1 mm

Commit message: BOM Fix
Realized I specified a 1206 resistor instead of 0805. Fixed the BOM. Also added an HTML exported BOM for easy reading.
Other:
- board text added: "Sega CD Back-up RAM Cart (4Mbit) v1.1 Designed by WindDrake with help from Officer_Skidmark Based on l_oliveira's original research github.com/WindDrake/SegaCD_Ramcart"
- board text removed: "Sega CD Back-up RAM Cart (4Mbit) v1.0 Designed by WindDrake with help from Officer_Skidmark Based on l_oliveira's original research github.com/WindDrake/SegaCD_Ramcart"

Commit message: 1.2 Overhaul
Changed SRAM, protection diode, protection resistor to fix battery lifetime problem. Added R2 to fix lack of sleep mode.
Parts:
- removed REF**: OSHW-Logo2_14.6x12mm_SilkScreen, Symbol:OSHW-Logo2_14.6x12mm_SilkScreen
- removed REF**: Symbol_CreativeCommonsPublicDomain_SilkScreenTop_Small, Symbol:Symbol_CreativeCommonsPublicDomain_SilkScreenTop_Small
- removed REF**: KiCad-Logo2_12mm_SilkScreen, Symbol:KiCad-Logo2_12mm_SilkScreen
- added R2: 10k, Resistor_SMD:R_0805_2012Metric_Pad1.20x1.40mm_HandSolder, F.Cu at (90.2, 146.6)
Connections:
- J1 pad A21: Net-(J1-PadA21) -> unconnected-(J1-PadA21)
- J1 pad A24: Net-(J1-PadA24) -> unconnected-(J1-PadA24)
- J1 pad A27: Net-(J1-PadA27) -> unconnected-(J1-PadA27)
- J1 pad A30: Net-(J1-PadA30) -> unconnected-(J1-PadA30)
- J1 pad B1: Net-(J1-PadB1) -> unconnected-(J1-PadB1)
- J1 pad B11: Net-(J1-PadB11) -> unconnected-(J1-PadB11)
- J1 pad B12: Net-(J1-PadB12) -> unconnected-(J1-PadB12)
- J1 pad B13: Net-(J1-PadB13) -> unconnected-(J1-PadB13)
- J1 pad B14: Net-(J1-PadB14) -> unconnected-(J1-PadB14)
- J1 pad B15: Net-(J1-PadB15) -> unconnected-(J1-PadB15)
- J1 pad B18: Net-(J1-PadB18) -> unconnected-(J1-PadB18)
- J1 pad B19: Net-(J1-PadB19) -> unconnected-(J1-PadB19)
- J1 pad B2: Net-(J1-PadB2) -> unconnected-(J1-PadB2)
- J1 pad B20: Net-(J1-PadB20) -> unconnected-(J1-PadB20)
- J1 pad B21: Net-(J1-PadB21) -> unconnected-(J1-PadB21)
- J1 pad B22: Net-(J1-PadB22) -> unconnected-(J1-PadB22)
- J1 pad B23: Net-(J1-PadB23) -> unconnected-(J1-PadB23)
- J1 pad B24: Net-(J1-PadB24) -> unconnected-(J1-PadB24)
- J1 pad B25: Net-(J1-PadB25) -> unconnected-(J1-PadB25)
- J1 pad B26: Net-(J1-PadB26) -> unconnected-(J1-PadB26)
- J1 pad B29: Net-(J1-PadB29) -> unconnected-(J1-PadB29)
- J1 pad B3: Net-(J1-PadB3) -> unconnected-(J1-PadB3)
- J1 pad B30: Net-(J1-PadB30) -> unconnected-(J1-PadB30)
- J1 pad B31: Net-(J1-PadB31) -> unconnected-(J1-PadB31)
- J1 pad B32: Net-(J1-PadB32) -> unconnected-(J1-PadB32)
- U4 pad 10: Net-(U4-Pad10) -> unconnected-(U4-Pad10)
- U4 pad 12: Net-(U4-Pad12) -> unconnected-(U4-Pad12)
- U4 pad 13: Net-(U4-Pad13) -> unconnected-(U4-Pad13)
- U4 pad 14: Net-(U4-Pad14) -> unconnected-(U4-Pad14)
- U4 pad 15: Net-(U4-Pad15) -> unconnected-(U4-Pad15)
- U5 pad 11: Net-(U5-Pad11) -> unconnected-(U5-Pad11)
- U6 pad 5: Net-(U6-Pad5) -> unconnected-(U6-Pad5)
- U6 pad 8: Net-(U6-Pad8) -> unconnected-(U6-Pad8)
- U6 pad 9: Net-(U6-Pad9) -> unconnected-(U6-Pad9)
Routing:
- net /SRCE: track 32.0 -> 66.0 mm, vias 3 -> 4
- net VBUS: track 17.0 -> 29.6 mm, vias 2 -> 3
- net Net-(BT1-PadP): track 72.5 -> 66.5 mm
- net +5V: track 291.4 -> 287.5 mm
- net GND: track 81.9 -> 80.8 mm, vias 51 -> 53
- net /A1: track 35.3 -> 36.3 mm
- net /A17: track 66.7 -> 66.0 mm
- net /A12: vias 2 -> 1
Other:
- net class Default removed
- board text added: "Sega CD Back-up RAM Cart (4Mbit) v1.2 Designed by WindDrake with help from Officer_Skidmark Based on l_oliveira's original research github.com/WindDrake/SegaCD_Ramcart"
- board text removed: "Sega CD Back-up RAM Cart (4Mbit) v1.1 Designed by WindDrake with help from Officer_Skidmark Based on l_oliveira's original research github.com/WindDrake/SegaCD_Ramcart"
